File: hardware/panel-stack/samplooler-panel-stack.kicad_pcb (KiCad board)
At the start: 2 copper layers, 94 x 94 mm, 36 parts, among them J1 To bottom board, J1 To top board, J2 MAX98357A (opt), J3 Qwiic I2C, J4 EXP A, J5 EXP B, SW1 EC11, 25 mm shaft, U1 ESP32-S3_SuperMini, U1 OLED 0.96in, U2 INMP441, U2 PCM5102A, U4 MPU6050, U5 KY-023

Commit message: Rev D boards, firmware and page changes (work in progress, before the launch cleanup)
Co-Authored-By: Claude Opus 5.5 <noreply@anthropic.com>
Parts:
- removed the JP1 at (82.7, 70.4)
- removed the JP2 at (80.2, 73.4)
- removed JP3: XSMT, Jumper:SolderJumper-3_P1.3mm_Open_RoundedPad1.0x1.5mm
- removed JP4: FMT, Jumper:SolderJumper-3_P1.3mm_Open_RoundedPad1.0x1.5mm
- U1: value OLED 0.96in -> OLED 0.96in (under); footprint samplooler:SSD1306_0.96in_I2C -> samplooler:SSD1306_0.96in_I2C_Under; moved to B.Cu
- U2: value INMP441 -> INMP441 (under); footprint samplooler:INMP441_Round -> samplooler:INMP441_Round_Under; moved to B.Cu
- U5: value KY-023 -> PS2 joystick (KY-023 part); footprint samplooler:KY-023_Joystick -> samplooler:PS2_Joystick
- moved U5 15.9 mm to (75.0, 80.6), turned to 180 degrees
Connections:
- U2 pad 10: /DAC_FMT -> GND
- U2 pad 7: /DAC_FLT -> GND
- U2 pad 8: /DAC_DEMP -> GND
- U2 pad 9: /DAC_XSMT -> /DAC_3V3
- U5 pad 1: GND -> +3V3
- U5 pad 2: +3V3 -> /JOY_X
- U5 pad 3: /JOY_X -> GND
- U5 pad 4: /JOY_Y -> +3V3
- U5 pad 5: /JOY_SW -> /JOY_Y
Routing:
- net /GPIO33: track 85.6 -> 36.9 mm, vias 6 -> 1
- net /ENC_B: track 77.2 -> 31.0 mm, vias 3 -> 2
- net +3V3: track 256.3 -> 213.2 mm, vias 3 -> 1
- net /ENC_A: track 74.0 -> 38.0 mm, vias 4 -> 3
- net /JOY_Y: track 69.8 -> 43.0 mm
- net /GPIO48: track 48.3 -> 26.5 mm, vias 1 -> 2
- net /I2S_WS: track 169.8 -> 191.4 mm, vias 0 -> 1
- net /GPIO47: track 45.0 -> 23.8 mm, vias 2 -> 1
- net /OLED_P1: track 30.3 -> 48.2 mm, vias 0 -> 1
- net /GPIO46: track 23.6 -> 40.9 mm
- net +5V: track 148.1 -> 165.3 mm
- net /GPIO15: track 31.3 -> 45.2 mm, vias 1 -> 0
- net /DAC_FMT: track 12.4 -> 0.00 mm
- net /DAC_3V3: track 20.8 -> 8.58 mm, vias 1 -> 0
- net /GPIO14: track 30.9 -> 42.8 mm
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Other:
- outline, holes or cut-outs redrawn
- board text added: "DAC: FLT DEMP FMT = L, XSMT = H"
- board text added: "J1 header goes on THIS side, pins down"
- board text added: "MIC: flush, sound hole up over the port"
- board text added: "OLED: header plastic on the glass side"
- board text added: "hold: freeze the tilt"
- board text added: "knob tap: menu turn: value"
- board text added: "rev D"
- board text added: "rev D 2026-10-15"
- board text added: "stack bottom rev D 2026-10-15"
- board text added: "stick hold down: record"
- board text removed: "1-2 = H 2-3 = L"
- board text removed: "DAC straps"
- board text removed: "DEMP"
- board text removed: "FLT"
- board text removed: "FMT"
- board text removed: "J1 header goes on THIS side,"
- board text removed: "XSMT"
- board text removed: "knob turn: value hold: record"
- board text removed: "open if set on"
- board text removed: "pins down"
- board text removed: "rev C"
- board text removed: "rev C 2026-09-28"
- board text removed: "stack bottom rev C 2026-09-28"
- board text removed: "stick click: tilt hold: menu"
- board text removed: "the DAC board"
