File: hardware/stack-bottom/samplooler-stack-bottom.kicad_sch (KiCad schematic)
At the start: 23 parts, among them J1 To top board, J2 MAX98357A (opt), J3 Qwiic I2C, J4 EXP A, J5 EXP B, SW1 EC11, 25 mm shaft, U1 ESP32-S3_SuperMini, U2 PCM5102A, U4 MPU6050, U5 KY-023

Commit message: Stack boards at 94 x 46 mm, one-piece JLC panels for the stack and the Mini + Filter
The stack's two boards shrink to 94 x 46 mm with the DAC straps under the
bottom board and both breakout rows in the middle, under the top board.
New hardware/gen/panel.py copies built boards onto one panel with 5 mm
tabs and mouse bites: the stack at 94 x 94 mm (panel-stack/), and the Mini
with the Samplooler Filter at 82 x 94 mm (panel-mini/), with their JLC zips,
BOM and CPL files and renders. kit.py checks router sessions for crossing
tracks of different nets before accepting them. hardware/README.md, CLAUDE.md
and the pcb-design skill describe the panels and the ordering settings.

Co-Authored-By: Claude Fable 5.1 <noreply@anthropic.com>
Connections:
- net +3V3: now also J4.14 (3V3), J5.12 (3V3); no longer J4.13 (3V3), J5.1 (3V3)
- net +5V: now also J5.14 (5V); no longer J5.3 (5V)
- net GND: now also J4.13 (GND), J5.11 (GND), J5.13 (GND); no longer J4.14 (GND), J5.2 (GND), J5.4 (GND)
- net GPIO14: now also J5.6 (14); no longer J4.5 (14)
- net GPIO15: now also J5.5 (15); no longer J4.6 (15)
- net GPIO16: now also J5.8 (16); no longer J4.7 (16)
- net GPIO17: now also J5.7 (17); no longer J4.8 (17)
- net GPIO18: now also J5.3 (18); no longer J4.4 (18)
- net GPIO21: now also J5.4 (21); no longer J4.3 (21)
- net GPIO33: now also J5.1 (33); no longer J4.2 (33)
- net GPIO34: now also J5.2 (34); no longer J4.1 (34)
- net GPIO35: now also J5.10 (35); no longer J4.9 (35)
- net GPIO36: now also J5.9 (36); no longer J4.10 (36)
- net GPIO37: now also J4.12 (37); no longer J4.11 (37)
- net GPIO38: now also J4.10 (38); no longer J4.12 (38)
- net GPIO39: now also J4.4 (39); no longer J5.11 (39)
- net GPIO40: now also J4.3 (40); no longer J5.12 (40)
- net GPIO41: now also J4.6 (41); no longer J5.9 (41)
- net GPIO42: now also J4.5 (42); no longer J5.10 (42)
- net GPIO43: now also J4.1 (43); no longer J5.13 (43)
- net GPIO44: now also J4.2 (44); no longer J5.14 (44)
- net GPIO45: now also J4.8 (45); no longer J5.7 (45)
- net GPIO46: now also J4.7 (46); no longer J5.8 (46)
- net GPIO47: now also J4.9 (47); no longer J5.5 (47)
- net GPIO48: now also J4.11 (48); no longer J5.6 (48)

Commit message: Rev D boards, firmware and page changes (work in progress, before the launch cleanup)
Co-Authored-By: Claude Opus 5.5 <noreply@anthropic.com>
Parts:
- removed JP1: FLT, Jumper:SolderJumper-3_P1.3mm_Open_RoundedPad1.0x1.5mm, symbol Jumper:SolderJumper_3_Open
- removed JP2: DEMP, Jumper:SolderJumper-3_P1.3mm_Open_RoundedPad1.0x1.5mm, symbol Jumper:SolderJumper_3_Open
- removed JP3: XSMT, Jumper:SolderJumper-3_P1.3mm_Open_RoundedPad1.0x1.5mm, symbol Jumper:SolderJumper_3_Open
- removed JP4: FMT, Jumper:SolderJumper-3_P1.3mm_Open_RoundedPad1.0x1.5mm, symbol Jumper:SolderJumper_3_Open
- U5: value KY-023 -> PS2 joystick (KY-023 part); footprint samplooler:KY-023_Joystick -> samplooler:PS2_Joystick; symbol samplooler:KY-023_Joystick -> samplooler:PS2_Joystick
Connections:
- net DAC_DEMP is gone; now on net GND: U2.8 (DEMP)
- net DAC_FLT is gone; now on net GND: U2.7 (FLT)
- net DAC_FMT is gone; now on net GND: U2.10 (FMT)
- net DAC_XSMT is gone; now on net DAC_3V3: U2.9 (XSMT)
- net +3V3: now also U5.1 (H1), U5.4 (V1); no longer U5.2 (+5V)
- net GND: now also U5.3 (H3), U5.6 (V3), U5.7 (SW1); no longer U5.1 (GND)
- net JOY_SW: now also U5.9 (SW2); no longer U5.5 (SW)
- net JOY_X: now also U5.2 (H2); no longer U5.3 (VRx)
- net JOY_Y: now also U5.5 (V2); no longer U5.4 (VRy)
- no-connect marks 7 -> 12
Other:
- note added: "DAC (GY-PCM5102, line out; FLT DEMP FMT low, XSMT high)"
- note added: "DAC control pins are tied here, no straps: FLT, DEMP, FMT to GND (normal filter, no de-emphasis, I2S), XSMT to A3V3, the module's own 3.3 V (unmuted). A floating FMT distorts at a touch. Matches the H1L-H4L bridges on the DAC board's back if they are set as usual (L L H L)."
- note added: "Joystick (the KY-023's PS2-style stick, no module board; press = record)"
- note added: "Joystick pots run from 3V3 (not 5V): the ESP32 ADC reads 0-3.3 V. The IMU's +X axis points at the nose (the USB / jack edge). AD0 to GND: address 0x68."
- note removed: "DAC (GY-PCM5102, line out)"
- note removed: "JP1-JP4 stand in for the H1L-H4L bridges on the back of the DAC board, out of reach once it is mounted. Leave them OPEN if those are set; otherwise FLT=L, DEMP=L, XSMT=H (unmute), FMT=L. H is DAC_3V3, the module's own 3.3 V regulator, never the board 3V3."
- note removed: "Joystick (KY-023)"
- note removed: "The joystick's "+5V" pin goes to 3V3: the ESP32 ADC reads 0-3.3 V. The IMU's +X axis points at the nose (the USB / jack edge). AD0 to GND: address 0x68."
- moved on the sheet: C1, C2, C3, H1, H2, H3, H4, J1, J2, J3, J4, J5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
