File: hardware/stack-top/samplooler-stack-top.kicad_sch (KiCad schematic)
At the start: 12 parts, among them J1 To bottom board, U1 OLED 0.96in, U2 INMP441

Commit message: Rev D boards, firmware and page changes (work in progress, before the launch cleanup)
Co-Authored-By: Claude Opus 5.5 <noreply@anthropic.com>
Parts:
- U1: value OLED 0.96in -> OLED 0.96in (under); footprint samplooler:SSD1306_0.96in_I2C -> samplooler:SSD1306_0.96in_I2C_Under; symbol samplooler:SSD1306_0.96in_I2C -> samplooler:SSD1306_0.96in_I2C_Under
- U2: value INMP441 -> INMP441 (under); footprint samplooler:INMP441_Round -> samplooler:INMP441_Round_Under; symbol samplooler:INMP441_Round -> samplooler:INMP441_Round_Under
Other:
- note added: "Microphone (INMP441, I2S; under the board, flush, through a 1.5 mm port)"
- note added: "OLED (SSD1306 0.96in, I2C 0x3C; under the board, through a window)"
- note added: "U1 and U2 hang under this board facing up. The OLED's header goes in from the glass side (plastic between glass side and board); the mic sits flush, sound hole over the port."
- note removed: "Microphone (INMP441, I2S, sound hole up)"
- note removed: "OLED (SSD1306 0.96in, I2C 0x3C)"
- moved on the sheet: C3, H1, H2, H3, H4, U2
